Commit message: Update: Changed gripper and moveit config

File: src/arm_description/urdf/my_panda.urdf (robot description, URDF)
Before this commit: robot panda, 12 links, 11 joints
Links:
- removed link panda_finger
- added link panda_leftfinger, mass 0.5; collision mesh filename=package://arm_description/meshes/collision/finger.stl; visual mesh filename=package://arm_description/meshes/visual/finger.dae
- added link panda_random
- added link panda_rightfinger, mass 0.5; collision mesh filename=package://arm_description/meshes/collision/finger.stl; visual mesh filename=package://arm_description/meshes/visual/finger.dae
Joints:
- removed joint panda_finger_joint
- added joint panda_finger_joint1: type prismatic, parent panda_hand, child panda_leftfinger, origin xyz=0 0 0.0584 rpy=0 0 0, axis 0 1 0, limit lower=0.0 upper=0.04 effort=40 velocity=0.2
- added joint panda_finger_joint2: type prismatic, parent panda_hand, child panda_rightfinger, origin xyz=0 0 0.0584 rpy=0 0 0, axis 0 -1 0, limit lower=0.0 upper=0.04 effort=40 velocity=0.2, mimic joint=panda_finger_joint1
- added joint panda_finger_joint2_mimic: type fixed, parent panda_hand, child panda_random

File: src/arm_description/urdf/panda_hand.xacro (robot description, xacro)
@@ -28,62 +28,64 @@
     </link>
     <!-- Left Finger Link -->
-    <link name="${ns}_finger_left">
+    <link name="${ns}_leftfinger">
       <visual>
-        <origin xyz="-0.02 0 0.02" rpy="0 0 0"/>
         <geometry>
-          <box size="0.01 0.04 0.04"/>
+          <mesh filename="package://arm_description/meshes/visual/finger.dae" />
         </geometry>
       </visual>
       <collision>
-        <origin xyz="-0.02 0 0.02" rpy="0 0 0"/>
         <geometry>
-          <box size="0.01 0.04 0.04"/>
+          <mesh filename="package://arm_description/meshes/collision/finger.stl" />
         </geometry>
       </collision>
       <inertial>
-        <origin xyz="0 0 0" rpy="0 0 0"/>
-        <mass value="0.02"/>
-        <inertia ixx="0.000001667" ixy="0.0" ixz="0.0" iyy="0.000001667" iyz="0.0" izz="0.000000667"/>
+        <origin xyz="0 0 0.32" />
+        <mass value="0.5" />
+        <inertia ixx="0.002" ixy="0" ixz="0" iyy="0.002" iyz="0" izz="0.002" />
       </inertial>
     </link>
     <!-- Right Finger Link -->
-    <link name="${ns}_finger_right">
+    <link name="${ns}_rightfinger">
       <visual>
-        <origin xyz="0.02 0 0.02" rpy="0 0 0"/>
+        <origin rpy="0 0 3.14159265359" xyz="0 0 0" />
         <geometry>
-          <box size="0.01 0.04 0.04"/>
+          <mesh filename="package://arm_description/meshes/visual/finger.dae" />
         </geometry>
       </visual>
       <collision>
-        <origin xyz="0.02 0 0.02" rpy="0 0 0"/>
+        <origin rpy="0 0 3.14159265359" xyz="0 0 0" />
         <geometry>
-          <box size="0.01 0.04 0.04"/>
+          <mesh filename="package://arm_description/meshes/collision/finger.stl" />
         </geometry>
       </collision>
       <inertial>
-        <origin xyz="0 0 0" rpy="0 0 0"/>
-        <mass value="0.02"/>
-        <inertia ixx="0.000001667" ixy="0.0" ixz="0.0" iyy="0.000001667" iyz="0.0" izz="0.000000667"/>
+        <origin xyz="0 0 0.32" />
+        <mass value="0.5" />
+        <inertia ixx="0.002" ixy="0" ixz="0" iyy="0.002" iyz="0" izz="0.002" />
       </inertial>
     </link>
     <!-- Left Finger Joint -->
-    <joint name="${ns}_finger_left_joint" type="revolute">
+    <joint name="${ns}_finger_joint1" type="prismatic">
       <parent link="${ns}_hand" />
-      <child link="${ns}_finger_left" />
-      <origin xyz="0 0 0.0584" rpy="0 0 0" />
-      <axis xyz="0 1 0"/>
-      <limit effort="20" lower="-0.25" upper="0.3390" velocity="0.2"/>
-      <dynamics damping="1.0"/>
+      <child link="${ns}_leftfinger" />
+      <origin rpy="0 0 0" xyz="0 0 0.0584" />
+      <axis xyz="0 1 0" />
+      <limit effort="40" lower="0.0" upper="0.04" velocity="0.2" />
     </joint>
     <!-- Right Finger Joint -->
-    <joint name="${ns}_finger_right_joint" type="revolute">
+    <joint name="${ns}_finger_joint2" type="prismatic">
       <parent link="${ns}_hand" />
-      <child link="${ns}_finger_right" />
-      <origin xyz="0 0 0.0584" rpy="0 0 0" />
-      <axis xyz="0 1 0"/>
-      <limit effort="20" lower="-0.3390" upper="0.25" velocity="0.2"/>
-      <dynamics damping="1.0"/>
-      <mimic joint="panda_finger_left_joint" multiplier="-1"/>
+      <child link="${ns}_rightfinger" />
+      <origin rpy="0 0 0" xyz="0 0 0.0584" />
+      <axis xyz="0 -1 0" />
+      <limit effort="40" lower="0.0" upper="0.04" velocity="0.2" />
+      <mimic joint="${ns}_finger_joint1" />
     </joint>
+    <!-- Dummy fixed joint and link to match the original structure -->
+    <joint name="${ns}_finger_joint2_mimic" type="fixed">
+      <parent link="${ns}_hand" />
+      <child link="${ns}_random" />
+    </joint>
+    <link name="${ns}_random"/>
   </xacro:macro>
 </robot>

File: src/my_panda_moveit_config/config/panda.ros2_control.xacro (robot description, xacro)
@@ -57,8 +57,8 @@
                 <state_interface name="velocity"/>
             </joint>
-            <joint name="panda_finger_left_joint">
+            <joint name="panda_finger_joint1">
                 <command_interface name="position"/>
                 <state_interface name="position">
-                  <param name="initial_value">${initial_positions['panda_finger_left_joint']}</param>
+                  <param name="initial_value">${initial_positions['panda_finger_joint1']}</param>
                 </state_interface>
                 <state_interface name="velocity"/>

File: src/my_panda_moveit_config/config/panda.urdf.xacro (robot description, xacro)
@@ -3,5 +3,5 @@
     <xacro:arg name="initial_positions_file" default="initial_positions.yaml" />
     <!-- Import panda urdf file -->
-    <xacro:include filename="$(find arm_description)/urdf/my_panda_new.urdf" />
+    <xacro:include filename="$(find arm_description)/urdf/my_panda.urdf" />
     <!-- Import control_xacro -->
     <xacro:include filename="panda.ros2_control.xacro" />
