Commit message: Update: modified moveit package

File: src/arm_description/urdf/manipulator.urdf.xacro (robot description, xacro)
@@ -9,4 +9,4 @@
   <xacro:panda_arm />
   <!-- call the hand macro-->
-  <xacro:panda_hand ns="panda" rpy="0 0 ${-pi/4}" connected_to="panda_link8" />
+  <xacro:panda_hand ns="panda" rpy="0 0 0" connected_to="panda_link8" />
 </robot>

File: src/arm_description/urdf/my_panda.urdf (robot description, URDF)
Before this commit: robot panda, 14 links, 13 joints
Joints:
- joint panda_hand_joint: origin xyz=0 0 0 rpy=0 0 -0.7853981633974483 -> xyz=0 0 0 rpy=0 0 0
- joint panda_joint6: origin xyz=0 0 0 rpy=1.5707963267948966 0 0 -> xyz=0 0 0 rpy=-1.5707963267948966 0 0

File: src/arm_description/urdf/panda_arm.xacro (robot description, xacro)
@@ -243,5 +243,5 @@
       <safety_controller k_position="100.0" k_velocity="40.0" soft_lower_limit="-0.0175"
         soft_upper_limit="3.7525" />
-      <origin rpy="${pi/2} 0 0" xyz="0 0 0" />
+      <origin rpy="${-pi/2} 0 0" xyz="0 0 0" />
       <parent link="${arm_id}_link5" />
       <child link="${arm_id}_link6" />
