Commit message: update:  pick-place s initial working

File: src/arm_description/urdf/panda.urdf (robot description, URDF)
Before this commit: robot panda, 12 links, 11 joints
Links:
- added link world
- link panda_hand: mass None -> 0.5
- link panda_leftfinger: mass None -> 0.5
- link panda_link0: mass None -> 50
- link panda_link1: mass None -> 0.5
- link panda_link2: mass None -> 0.5
- link panda_link3: mass None -> 0.5
- link panda_link4: mass None -> 0.5
- link panda_link5: mass None -> 0.5
- link panda_link6: mass None -> 0.5
- link panda_link7: mass None -> 0.5
- link panda_rightfinger: mass None -> 0.5
Joints:
- added joint connect_root_and_world: type fixed, parent world, child panda_link0, origin xyz=0 0 0 rpy=0 0 0
- joint panda_finger_joint1: limit lower=0.0 upper=0.04 effort=20 velocity=0.2 -> lower=0.0 upper=0.04 effort=40 velocity=0.2; origin xyz=0 0 0.0584 rpy=0 0 0 -> xyz=0.0 0.0 0.0584 rpy=0.0 0.0 0.0
- joint panda_finger_joint2: limit lower=0.0 upper=0.04 effort=20 velocity=0.2 -> lower=0.0 upper=0.04 effort=40 velocity=0.2; origin xyz=0 0 0.0584 rpy=0 0 0 -> xyz=0.0 0.0 0.0584 rpy=0.0 0.0 0.0

File: src/panda_moveit_config/config/panda.ros2_control.xacro (robot description, xacro)
@@ -14,6 +14,6 @@
                 </xacro:if> -->
               <plugin>topic_based_ros2_control/TopicBasedSystem</plugin>
-              <param name="joint_commands_topic">/isaac_joint_commands</param>
-              <param name="joint_states_topic">/isaac_joint_states</param>
+              <param name="joint_commands_topic">/joint_commands</param>
+              <param name="joint_states_topic">/joint_states</param>
             </hardware>
             <joint name="panda_joint1">

File: src/panda_moveit_config/config/panda_hand.ros2_control.xacro (robot description, xacro)
@@ -13,6 +13,6 @@
                 </xacro:if> -->
                 <plugin>topic_based_ros2_control/TopicBasedSystem</plugin>
-                <param name="joint_commands_topic">/isaac_joint_commands</param>
-                <param name="joint_states_topic">/isaac_joint_states</param>
+                <param name="joint_commands_topic">/joint_commands</param>
+                <param name="joint_states_topic">/joint_states</param>
             </hardware>
             <joint name="panda_finger_joint1">
